File: ESPFirmwareV2/Circuit/HomeSecurity-Circuits/HomeSecurity-Circuits.kicad_sch (KiCad schematic)
At the start: 3 parts

Commit message: fix: use pdMS_TO_TICKS for UART timeout, add vTaskDelay to main loop
- Replace raw integer 100 with pdMS_TO_TICKS(100) in uart_read_bytes
- Add vTaskDelay(10) to main loop to yield FreeRTOS task
- Update VSCode COM ports: Station 101→1101, AP 110→10
- Rename KiCad footprint library customespfootprint → HomeSecurity-Proj
- Rewrite CLAUDE.md (Station) with structured docs and debugging discipline
- Delete CLAUDE.md (AP)
Parts:
- U1, U2: footprint customespfootprint:esp32wroom -> HomeSecurity-Proj:esp32wroom
- U3: footprint customespfootprint:ili9488 -> HomeSecurity-Proj:ili9488
Changed lines of the file:
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@@
 			)
 		)
-		(property "Footprint" "customespfootprint:esp32wroom"
+		(property "Footprint" "HomeSecurity-Proj:esp32wroom"
 			(at 179.07 81.28 0)
 			(effects
@@
 			)
 		)
-		(property "Footprint" "customespfootprint:ili9488"
+		(property "Footprint" "HomeSecurity-Proj:ili9488"
 			(at 153.67 138.43 0)
 			(effects
@@
 			)
 		)
-		(property "Footprint" "customespfootprint:esp32wroom"
+		(property "Footprint" "HomeSecurity-Proj:esp32wroom"
 			(at 105.41 81.28 0)
 			(effects
